Commit message: make rollerwalker in gazebo

File: src/rollerwalker_sim/xacro/rollerwalker.xacro (robot description, xacro)
@@ -315,14 +315,4 @@
             <!-- <limit lower="-1.79769e+308" upper="1.79769e+308" effort="0" velocity="0"/> -->
         </joint>
-        <!-- ジョイント3のトランスミッション -->
-        <transmission name="wheel_trans" >
-            <type>transmission_interface/SimpleTransmission</type>
-            <actuator name="$wheel_motor">
-                <mechanicalReduction>1</mechanicalReduction>
-            </actuator>
-            <joint name="link_4_${leg_posi}_to_wheel_${leg_posi}">
-                <hardwareInterface>hardware_interface/PositionJointInterface</hardwareInterface>
-            </joint>
-         </transmission>
         <!-- ホイールの描画 -->
         <link name = "wheel_${leg_posi}">
@@ -382,4 +372,14 @@
             </joint>
          </transmission>
+        <!-- ホイールのトランスミッション  -->
+        <transmission name="wheel_trans" >
+            <type>transmission_interface/SimpleTransmission</type>
+            <actuator name="$wheel_motor">
+                <mechanicalReduction>1</mechanicalReduction>
+            </actuator>
+            <joint name="link_4_${leg_posi}_to_wheel_${leg_posi}">
+                <hardwareInterface>hardware_interface/PositionJointInterface</hardwareInterface>
+            </joint>
+        </transmission>
     </xacro:macro>
     <!-- 本体の描画 -->

Commit message: create teleop keyboard

File: src/rollerwalker_sim/xacro/rollerwalker.xacro (robot description, xacro)
@@ -17,4 +17,16 @@
     </material>
     <!-- 各パラメータ -->
+    <!-- 各リンクの重量設定 -->
+    <xacro:property name="total_mass" value="23.8" />
+    <xacro:property name="body_mass" value="${total_mass*2/3}" />
+    <xacro:property name="leg_mass" value="${total_mass/3}" />
+    <xacro:property name="joint_1_mass" value="0.1" />
+    <xacro:property name="joint_2_mass" value="0.1" />
+    <xacro:property name="joint_3_mass" value="0.1" />
+    <xacro:property name="joint_4_mass" value="0.1" />
+    <xacro:property name="link_2_mass" value="${leg_mass/2}" />
+    <xacro:property name="link_3_mass" value="${leg_mass/3}" />
+    <xacro:property name="link_4_mass" value="${leg_mass/12}" />
+    <xacro:property name="wheel_mass" value="${leg_mass/12}" />
     <!-- ボディ関連 -->
     <xacro:property name="body_z" value="0.2" /> <!-- ボディの高さ -->
@@ -22,5 +34,4 @@
     <xacro:property name="body_width" value="0.29" />
     <xacro:property name="body_thickness" value="0.123" />
-    <xacro:property name="body_mass" value="23.8" />
     <!-- ボディーのイナーシャ -->
     <xacro:property name="I_body_xx" value="${1/12*body_mass*(body_thickness*body_thickness + body_width*body_width)}" />    <!--1/12m(h^2+d^2)-->
@@ -34,5 +45,4 @@
     <xacro:property name="wheel_radius" value="0.035" />
     <xacro:property name="wheel_thickness" value="0.024" />
-    <xacro:property name="wheel_mass" value="0.1" />
     <!-- タイヤのイナーシャ -->
     <xacro:property name="I_wheel_xx" value="${wheel_mass*(wheel_radius * wheel_radius/4 + wheel_thickness * wheel_thickness / 12)}" />     <!--M(R^2/4+h^2/12)-->
@@ -42,5 +52,4 @@
     <xacro:property name="joint_1_radius" value="0.05" />
     <xacro:property name="joint_1_thickness" value="0.1" />
-    <xacro:property name="joint_1_mass" value="0.1" />
     <!-- ジョイント1のイナーシャ -->
     <xacro:property name="I_joint_1_xx" value="${joint_1_mass*(joint_1_radius * joint_1_radius/4 + joint_1_thickness * joint_1_thickness / 12)}" />     <!--M(R^2/4+h^2/12)-->
@@ -50,5 +59,4 @@
     <xacro:property name="joint_2_radius" value="0.05" />
     <xacro:property name="joint_2_thickness" value="0.060" />
-    <xacro:property name="joint_2_mass" value="0.1" />
     <!-- ジョイント2のイナーシャ -->
     <xacro:property name="I_joint_2_xx" value="${joint_2_mass*(joint_2_radius * joint_2_radius/4 + joint_2_thickness * joint_2_thickness / 12)}" />     <!--M(R^2/4+h^2/12)-->
@@ -58,5 +66,4 @@
     <xacro:property name="joint_3_radius" value="0.04" />
     <xacro:property name="joint_3_thickness" value="0.05" />
-    <xacro:property name="joint_3_mass" value="0.1" />
     <!-- ジョイント3のイナーシャ -->
     <xacro:property name="I_joint_3_xx" value="${joint_3_mass*(joint_3_radius * joint_3_radius/4 + joint_3_thickness * joint_3_thickness / 12)}" />     <!--M(R^2/4+h^2/12)-->
@@ -66,5 +73,4 @@
     <xacro:property name="joint_4_radius" value="0.02" />
     <xacro:property name="joint_4_thickness" value="0.044" />
-    <xacro:property name="joint_4_mass" value="0.1" />
     <!-- ジョイント4のイナーシャ -->
     <xacro:property name="I_joint_4_xx" value="${joint_4_mass*(joint_4_radius * joint_4_radius/4 + joint_4_thickness * joint_4_thickness / 12)}" />     <!--M(R^2/4+h^2/12)-->
@@ -79,5 +85,4 @@
     <xacro:property name="link_2_y" value="0.055" />
     <xacro:property name="link_2_z" value="0.09" />
-    <xacro:property name="link_2_mass" value="0.1" />
     <!-- リンク2のイナーシャ -->
     <xacro:property name="I_link_2_xx" value="${1/12*link_2_mass*(link_2_y*link_2_y + link_2_z*link_2_z)}" />   <!--1/12m(h^2+d^2)-->
@@ -88,5 +93,4 @@
     <xacro:property name="link_3_y" value="0.045" />
     <xacro:property name="link_3_z" value="0.049" />
-    <xacro:property name="link_3_mass" value="0.1" />
     <!-- リンク3のイナーシャ -->
     <xacro:property name="I_link_3_xx" value="${1/12*link_3_mass*(link_3_y*link_3_y + link_3_z*link_3_z)}" />   <!--1/12m(h^2+d^2)-->
@@ -97,5 +101,4 @@
     <xacro:property name="link_4_y" value="0.043" />
     <xacro:property name="link_4_z" value="0.031" />
-    <xacro:property name="link_4_mass" value="0.1" />
     <!-- リンク4のイナーシャ -->
     <xacro:property name="I_link_4_xx" value="${1/12*link_4_mass*(link_4_y*link_4_y + link_4_z*link_4_z)}" />   <!--1/12m(h^2+d^2)-->
