Commit message: change to effort control

File: src/rollerwalker_sim/xacro/include/leg_macro.xacro (robot description, xacro)
@@ -52,4 +52,6 @@
         <gazebo reference="joint_1_${leg_posi}">
             <material>Gazebo/Blue</material>
+            <!-- <kp value="${kp}" /> -->
+            <!-- <kd value="10" /> -->
         </gazebo>
         <!-- ジョイント１とジョイント２の設定 -->
@@ -85,4 +87,6 @@
         <gazebo reference="joint_2_${leg_posi}">
             <material>Gazebo/Green</material>
+            <!-- <kp value="${kp}" /> -->
+            <!-- <kd value="10" /> -->
         </gazebo>
         <!-- ジョイント２とリンク２の設定 -->
@@ -150,4 +154,6 @@
         <gazebo reference="joint_3_${leg_posi}">
             <material>Gazebo/Yellow</material>
+            <!-- <kp value="${kp}" /> -->
+            <!-- <kd value="10" /> -->
         </gazebo>
         <!-- ジョイント3とリンク3の設定 -->
@@ -181,4 +187,6 @@
         <gazebo reference="link_3_${leg_posi}">
             <material>Gazebo/White</material>
+            <!-- <kp value="${kp}" /> -->
+            <!-- <kd value="10" /> -->
         </gazebo>
         <!-- リンク3とジョイント4の設定 -->
@@ -214,4 +222,6 @@
         <gazebo reference="joint_4_${leg_posi}">
             <material>Gazebo/Yellow</material>
+            <!-- <kp value="${kp}" /> -->
+            <!-- <kd value="10" /> -->
         </gazebo>
         <!-- ジョイント4とリンク4の描画 -->
@@ -245,4 +255,6 @@
         <gazebo reference="link_4_${leg_posi}">
             <material>Gazebo/Red</material>
+            <!-- <kp value="${kp}" /> -->
+            <!-- <kd value="10" /> -->
         </gazebo>
         <!-- リンク4とホイールの設定 -->
@@ -280,4 +292,6 @@
             <mu1>${mu_1}</mu1>
             <mu2>${mu_2}</mu2>
+            <!-- <kp value="${kp}" /> -->
+            <!-- <kd value="10" /> -->
         </gazebo>
         <!-- トランスミッション -->
@@ -288,5 +302,5 @@
             </actuator>
             <joint name="body_to_joint_1_${leg_posi}">
-                <hardwareInterface>hardware_interface/PositionJointInterface</hardwareInterface>
+                <hardwareInterface>hardware_interface/EffortJointInterface</hardwareInterface>
             </joint>
         </transmission>
@@ -298,5 +312,5 @@
             </actuator>
             <joint name="joint_1_${leg_posi}_to_joint_2_${leg_posi}">
-                <hardwareInterface>hardware_interface/PositionJointInterface</hardwareInterface>
+                <hardwareInterface>hardware_interface/EffortJointInterface</hardwareInterface>
             </joint>
         </transmission>
@@ -308,5 +322,5 @@
             </actuator>
             <joint name="link_2_${leg_posi}_to_joint_3_${leg_posi}">
-                <hardwareInterface>hardware_interface/PositionJointInterface</hardwareInterface>
+                <hardwareInterface>hardware_interface/EffortJointInterface</hardwareInterface>
             </joint>
          </transmission>
@@ -318,5 +332,5 @@
             </actuator>
             <joint name="link_3_${leg_posi}_to_joint_4_${leg_posi}">
-                <hardwareInterface>hardware_interface/PositionJointInterface</hardwareInterface>
+                <hardwareInterface>hardware_interface/EffortJointInterface</hardwareInterface>
             </joint>
          </transmission>
@@ -328,5 +342,5 @@
             </actuator>
             <joint name="link_4_${leg_posi}_to_wheel_${leg_posi}">
-                <hardwareInterface>hardware_interface/PositionJointInterface</hardwareInterface>
+                <hardwareInterface>hardware_interface/EffortJointInterface</hardwareInterface>
             </joint>
         </transmission>

File: src/rollerwalker_sim/xacro/include/rollerwalker_macro.xacro (robot description, xacro)
@@ -19,6 +19,6 @@
     <!-- 各リンクの重量設定 -->
     <xacro:property name="total_mass" value="23.8" />
-    <xacro:property name="body_mass" value="${total_mass*2/3}" />
-    <xacro:property name="leg_mass" value="${total_mass/3}" />
+    <xacro:property name="body_mass" value="${total_mass/3}" />
+    <xacro:property name="leg_mass" value="${total_mass*2/3}" />
     <xacro:property name="joint_1_mass" value="1.0" />
     <xacro:property name="joint_2_mass" value="1.0" />
@@ -77,7 +77,4 @@
     <xacro:property name="I_joint_4_yy" value="${joint_4_mass*(joint_4_radius * joint_4_radius/4 + joint_4_thickness * joint_4_thickness / 12)}" />     <!--M(R^2/4+h^2/12)-->
     <xacro:property name="I_joint_4_zz" value="${joint_4_mass* joint_4_radius * joint_4_radius/2}" />                                                  <!--1/2MR^2-->
-    <!-- 摩擦力 -->
-    <xacro:property name="mu_1" value="0.417" />
-    <xacro:property name="mu_2" value="0.0264" />
     <!-- 各足の長さはlink_n_xの値を変えれば良い -->
     <!-- リンク2関連 -->
@@ -114,3 +111,10 @@
     <xacro:property name="joint_4_to_link_4_damping" value="0.1" />   <!-- ジョイント4からリンク4のダンピング係数 -->
     <xacro:property name="link_4_to_wheel_damping" value="0.1" />   <!-- リンク4からホイールのダンピング係数 -->
+        <!-- 摩擦力 -->
+    <xacro:property name="mu_1" value="0.417" />
+    <xacro:property name="mu_2" value="0.0264" />
+    <xacro:property name="mu_1" value="0.417" />
+    <xacro:property name="mu_2" value="0.0264" />
+    <!-- めり込み係数 -->
+    <xacro:property name="kp" value="100000" />
 </robot>

Commit message: change to effort contorl

File: src/rollerwalker_sim/xacro/include/leg_macro.xacro (robot description, xacro)
@@ -11,20 +11,20 @@
             <xacro:if value="${leg_posi=='lf'}">
                 <origin xyz="${body_length/2 - joint_1_radius/2} ${body_width/2 - joint_1_radius/2} 0.0" rpy="0 0 0"/>
-                <limit lower="0.2" upper="3" effort="100" velocity="100"/>
+                <limit lower="0.2" upper="3" effort="${effort_limit}" velocity="100"/>
             </xacro:if>
             <!-- lr -->
             <xacro:if value="${leg_posi=='lr'}">
                 <origin xyz="${-(body_length/2 - joint_1_radius/2)} ${body_width/2 - joint_1_radius/2} 0.0" rpy="0 0 0"/>
-                <limit lower="0.2" upper="3" effort="100" velocity="100"/>
+                <limit lower="0.2" upper="3" effort="${effort_limit}" velocity="100"/>
             </xacro:if>
             <!-- rr -->
             <xacro:if value="${leg_posi=='rr'}">
                 <origin xyz="${-(body_length/2 - joint_1_radius/2)} ${-(body_width/2 - joint_1_radius/2)} 0.0" rpy="0 0 0"/>
-                <limit lower="-3" upper="-0.2" effort="100" velocity="100"/>
+                <limit lower="-3" upper="-0.2" effort="${effort_limit}" velocity="100"/>
             </xacro:if>
             <!-- rf -->
             <xacro:if value="${leg_posi=='rf'}">
                 <origin xyz="${body_length/2 - joint_1_radius/2} ${-(body_width/2 - joint_1_radius/2)} 0.0" rpy="0 0 0"/>
-                <limit lower="-3" upper="-0.2" effort="100" velocity="100"/>
+                <limit lower="-3" upper="-0.2" effort="${effort_limit}" velocity="100"/>
             </xacro:if>
             <dynamics damping="${body_to_joint_1_damping}"/>
@@ -62,5 +62,5 @@
             <origin rpy="1.57070 0 0" xyz="0 0 0"/>
             <dynamics damping="${joint_1_to_joint_2_damping}"/>
-            <limit lower="-1.5" upper="1.5" effort="100" velocity="100"/>
+            <limit lower="-1.5" upper="1.5" effort="${effort_limit}" velocity="100"/>
         </joint>
         <!-- ジョイント２の描画 -->
@@ -129,5 +129,5 @@
             <origin rpy="1.57070 0 0" xyz="${link_2_x} 0 0"/>
             <dynamics damping="${link_2_to_joint_3_damping}"/>
-            <limit lower="-2.0" upper="1.5" effort="100" velocity="100"/>
+            <limit lower="-2.0" upper="1.5" effort="${effort_limit}" velocity="100"/>
         </joint>
         <!-- ジョイント3の描画 -->
@@ -197,5 +197,5 @@
             <origin rpy="1.57070 0 0" xyz="${link_3_x} 0 0"/>
             <dynamics damping="${link_3_to_joint_4_damping}"/>
-            <limit lower="-2.0" upper="1.5" effort="100" velocity="100"/>
+            <limit lower="-2.0" upper="1.5" effort="${effort_limit}" velocity="100"/>
         </joint>
         <!-- ジョイント4の描画 -->
@@ -292,4 +292,5 @@
             <mu1>${mu_1}</mu1>
             <mu2>${mu_2}</mu2>
+            <!-- <fdir>0 0 1</fdir> -->
             <!-- <kp value="${kp}" /> -->
             <!-- <kd value="10" /> -->
@@ -342,5 +343,5 @@
             </actuator>
             <joint name="link_4_${leg_posi}_to_wheel_${leg_posi}">
-                <hardwareInterface>hardware_interface/EffortJointInterface</hardwareInterface>
+                <hardwareInterface>hardware_interface/VelocityJointInterface</hardwareInterface>
             </joint>
         </transmission>

File: src/rollerwalker_sim/xacro/include/rollerwalker_macro.xacro (robot description, xacro)
@@ -103,18 +103,20 @@
     <xacro:property name="I_link_4_zz" value="${1/12*link_4_mass*(link_4_x*link_4_x + link_4_y*link_4_y)}" />   <!--1/12m(w^2+d^2)-->
     <!-- ジョイントのダンピング係数 -->
-    <xacro:property name="body_to_joint_1_damping" value="0.1" />   <!-- ボディーからジョイント1のダンピング係数 -->
+    <xacro:property name="body_to_joint_1_damping"    value="0.1" />   <!-- ボディーからジョイント1のダンピング係数 -->
     <xacro:property name="joint_1_to_joint_2_damping" value="0.1" />   <!-- ジョイント1からジョイント2のダンピング係数 -->
-    <xacro:property name="joint_2_to_link_2_damping" value="0.1" />   <!-- ジョイント2からリンク2のダンピング係数 -->
-    <xacro:property name="link_2_to_joint_3_damping" value="0.1" />   <!-- リンク2からジョイント3のダンピング係数 -->
-    <xacro:property name="joint_3_to_link_3_damping" value="0.1" />   <!-- ジョイント3からリンク3のダンピング係数 -->
-    <xacro:property name="link_3_to_joint_4_damping" value="0.1" />   <!-- リンク3からジョイント4のダンピング係数 -->
-    <xacro:property name="joint_4_to_link_4_damping" value="0.1" />   <!-- ジョイント4からリンク4のダンピング係数 -->
-    <xacro:property name="link_4_to_wheel_damping" value="0.1" />   <!-- リンク4からホイールのダンピング係数 -->
+    <xacro:property name="joint_2_to_link_2_damping"  value="0.1" />   <!-- ジョイント2からリンク2のダンピング係数 -->
+    <xacro:property name="link_2_to_joint_3_damping"  value="0.1" />   <!-- リンク2からジョイント3のダンピング係数 -->
+    <xacro:property name="joint_3_to_link_3_damping"  value="0.1" />   <!-- ジョイント3からリンク3のダンピング係数 -->
+    <xacro:property name="link_3_to_joint_4_damping"  value="0.1" />   <!-- リンク3からジョイント4のダンピング係数 -->
+    <xacro:property name="joint_4_to_link_4_damping"  value="0.1" />   <!-- ジョイント4からリンク4のダンピング係数 -->
+    <xacro:property name="link_4_to_wheel_damping"    value="0.1" />   <!-- リンク4からホイールのダンピング係数 -->
         <!-- 摩擦力 -->
+    <!-- <xacro:property name="mu_1" value="0.417" />
+    <xacro:property name="mu_2" value="0.0264" />    -->
     <xacro:property name="mu_1" value="0.417" />
-    <xacro:property name="mu_2" value="0.0264" />
-    <xacro:property name="mu_1" value="0.417" />
-    <xacro:property name="mu_2" value="0.0264" />
+    <xacro:property name="mu_2" value="0.417" />
     <!-- めり込み係数 -->
     <xacro:property name="kp" value="100000" />
+    <!-- effort_limit -->
+    <xacro:property name="effort_limit" value="100000" />
 </robot>

Commit message: delete link_joint

File: src/rollerwalker_sim/xacro/include/leg_macro.xacro (robot description, xacro)
@@ -4,7 +4,7 @@
     <xacro:macro name="leg_macro" params="leg_posi">
         <!-- ジョイント1-->
-        <joint name="body_to_joint_1_${leg_posi}" type="revolute">
+        <joint name="joint_1_${leg_posi}" type="revolute">
             <parent link="body"/>
-            <child  link="joint_1_${leg_posi}"/>
+            <child  link="joint_1_link_${leg_posi}"/>
             <axis xyz="0 0 1"/>
             <!-- lf -->
@@ -28,7 +28,7 @@
                 <limit lower="-3" upper="-0.2" effort="${effort_limit}" velocity="100"/>
             </xacro:if>
-            <dynamics damping="${body_to_joint_1_damping}"/>
-        </joint>
-        <link name = "joint_1_${leg_posi}">
+            <dynamics damping="${joint_1_damping}"/>
+        </joint>
+        <link name = "joint_1_link_${leg_posi}">
             <inertial>
                 <mass value="${joint_1_mass}"/>
@@ -50,51 +50,17 @@
             </collision>
         </link>
-        <gazebo reference="joint_1_${leg_posi}">
+        <gazebo reference="joint_1_link_${leg_posi}">
             <material>Gazebo/Blue</material>
             <!-- <kp value="${kp}" /> -->
             <!-- <kd value="10" /> -->
         </gazebo>
-        <!-- ジョイント１とジョイント２の設定 -->
-        <joint name="joint_1_${leg_posi}_to_joint_2_${leg_posi}" type="revolute">
-            <axis xyz="0 0 1"/>
-            <parent link="joint_1_${leg_posi}"/>
-            <child  link="joint_2_${leg_posi}"/>
-            <origin rpy="1.57070 0 0" xyz="0 0 0"/>
+        <!-- ジョイント２の設定 -->
+        <joint name="joint_2_${leg_posi}" type="revolute">
+            <axis xyz="0 -1 0"/>
+            <parent link="joint_1_link_${leg_posi}"/>
+            <child  link="link_2_${leg_posi}"/>
+            <origin rpy="0 0 0" xyz="0 0 0"/>
             <dynamics damping="${joint_1_to_joint_2_damping}"/>
             <limit lower="-1.5" upper="1.5" effort="${effort_limit}" velocity="100"/>
-        </joint>
-        <!-- ジョイント２の描画 -->
-        <link name = "joint_2_${leg_posi}">
-            <inertial>
-                <mass value="${joint_2_mass}"/>
-                <origin xyz="${joint_1_radius/2} 0 0.0" rpy="0 0 0"/>
-                <inertia ixx="${I_joint_2_xx}" ixy="0.0" ixz="0.0" iyy="${I_joint_2_yy}" iyz="0.0" izz="${I_joint_2_zz}"/>
-            </inertial>
-            <visual>
-                <geometry>
-                    <cylinder radius="${joint_2_radius}" length="${joint_2_thickness}"/>
-                </geometry>
-                <origin xyz="${joint_1_radius/2} 0 0.0" rpy="0 0 0"/>
-                <material name = "green"/>
-            </visual>
-            <collision>
-                <origin xyz="${joint_1_radius/2} 0 0.0" rpy="0 0 0"/>
-                <geometry>
-                    <cylinder radius="${joint_2_radius}" length="${joint_2_thickness}"/>
-                </geometry>
-            </collision>
-        </link>
-        <gazebo reference="joint_2_${leg_posi}">
-            <material>Gazebo/Green</material>
-            <!-- <kp value="${kp}" /> -->
-            <!-- <kd value="10" /> -->
-        </gazebo>
-        <!-- ジョイント２とリンク２の設定 -->
-        <joint name="joint_2_${leg_posi}_to_link_2_${leg_posi}" type="fixed">
-            <axis xyz="0 0 1"/>
-            <parent link="joint_2_${leg_posi}"/>
-            <child  link="link_2_${leg_posi}"/>
-            <dynamics damping="${joint_2_to_link_2_damping}"/>
-            <origin rpy="-1.57070 0 0" xyz="0 0 0"/>
         </joint>
         <!-- リンク2の描画 -->
@@ -122,46 +88,12 @@
             <material>Gazebo/White</material>
         </gazebo>
-        <!-- リンク2とジョイント3の設定 -->
-        <joint name="link_2_${leg_posi}_to_joint_3_${leg_posi}" type="revolute">
-            <axis xyz="0 0 1"/>
+        <!-- ジョイント3の設定 -->
+        <joint name="joint_3_${leg_posi}" type="revolute">
+            <axis xyz="0 -1 0"/>
             <parent link="link_2_${leg_posi}"/>
-            <child  link="joint_3_${leg_posi}"/>
-            <origin rpy="1.57070 0 0" xyz="${link_2_x} 0 0"/>
+            <child  link="link_3_${leg_posi}"/>
+            <origin rpy="0 0 0" xyz="${link_2_x} 0 0"/>
             <dynamics damping="${link_2_to_joint_3_damping}"/>
             <limit lower="-2.0" upper="1.5" effort="${effort_limit}" velocity="100"/>
-        </joint>
-        <!-- ジョイント3の描画 -->
-        <link name = "joint_3_${leg_posi}">
-            <inertial>
-                <mass value="${joint_3_mass}"/>
-                <origin xyz="0 0 0.0" rpy="0 0 0"/>
-                <inertia ixx="${I_joint_3_xx}" ixy="0.0" ixz="0.0" iyy="${I_joint_3_yy}" iyz="0.0" izz="${I_joint_3_zz}"/>
-            </inertial>
-            <visual>
-                <geometry>
-                    <cylinder radius="${joint_3_radius}" length="${joint_3_thickness}"/>
-                </geometry>
-                <origin xyz="0 0 0.0" rpy="0 0 0"/>
-                <material name = "yellow"/>
-            </visual>
-            <collision>
-                <origin xyz="0 0 0.0" rpy="0 0 0"/>
-                <geometry>
-                    <cylinder radius="${joint_3_radius}" length="${joint_3_thickness}"/>
-                </geometry>
-            </collision>
-        </link>
-        <gazebo reference="joint_3_${leg_posi}">
-            <material>Gazebo/Yellow</material>
-            <!-- <kp value="${kp}" /> -->
-            <!-- <kd value="10" /> -->
-        </gazebo>
-        <!-- ジョイント3とリンク3の設定 -->
-        <joint name="joint_3_${leg_posi}_to_link_3_${leg_posi}" type="fixed">
-            <axis xyz="0 0 1"/>
-            <parent link="joint_3_${leg_posi}"/>
-            <child  link="link_3_${leg_posi}"/>
-            <dynamics damping="${joint_3_to_link_3_damping}"/>
-            <origin rpy="-1.57070 0 0" xyz="0 0 0"/>
         </joint>
         <link name = "link_3_${leg_posi}">
@@ -190,46 +122,12 @@
             <!-- <kd value="10" /> -->
         </gazebo>
-        <!-- リンク3とジョイント4の設定 -->
-        <joint name="link_3_${leg_posi}_to_joint_4_${leg_posi}" type="revolute">
-            <axis xyz="0 0 1"/>
+        <!-- ジョイント4の設定 -->
+        <joint name="joint_4_${leg_posi}" type="revolute">
+            <axis xyz="0 -1 0"/>
             <parent link="link_3_${leg_posi}"/>
-            <child  link="joint_4_${leg_posi}"/>
-            <origin rpy="1.57070 0 0" xyz="${link_3_x} 0 0"/>
+            <child  link="link_4_${leg_posi}"/>
+            <origin rpy="0 0 0" xyz="${link_3_x} 0 0"/>
             <dynamics damping="${link_3_to_joint_4_damping}"/>
             <limit lower="-2.0" upper="1.5" effort="${effort_limit}" velocity="100"/>
-        </joint>
-        <!-- ジョイント4の描画 -->
-        <link name = "joint_4_${leg_posi}">
-            <inertial>
-                <mass value="${joint_4_mass}"/>
-                <origin xyz="0 0 0.0" rpy="0 0 0"/>
-                <inertia ixx="${I_joint_4_xx}" ixy="0.0" ixz="0.0" iyy="${I_joint_4_yy}" iyz="0.0" izz="${I_joint_4_zz}"/>
-            </inertial>
-            <visual>
-                <geometry>
-                    <cylinder radius="${joint_4_radius}" length="${joint_4_thickness}"/>
-                </geometry>
-                <origin xyz="0 0 0.0" rpy="0 0 0"/>
-                <material name = "yellow"/>
-            </visual>
-            <collision>
-                <origin xyz="0 0 0.0" rpy="0 0 0"/>
-                <geometry>
-                    <cylinder radius="${joint_4_radius}" length="${joint_4_thickness}"/>
-                </geometry>
-            </collision>
-        </link>
-        <gazebo reference="joint_4_${leg_posi}">
-            <material>Gazebo/Yellow</material>
-            <!-- <kp value="${kp}" /> -->
-            <!-- <kd value="10" /> -->
-        </gazebo>
-        <!-- ジョイント4とリンク4の描画 -->
-        <joint name="joint_4_${leg_posi}_to_link_4_${leg_posi}" type="fixed">
-            <axis xyz="0 0 1"/>
-            <parent link="joint_4_${leg_posi}"/>
-            <child  link="link_4_${leg_posi}"/>
-            <origin rpy="-1.57070 0 0" xyz="0 0 0"/>
-            <dynamics damping="${joint_4_to_link_4_damping}"/>
         </joint>
         <link name = "link_4_${leg_posi}">
@@ -292,5 +190,5 @@
             <mu1>${mu_1}</mu1>
             <mu2>${mu_2}</mu2>
-            <!-- <fdir>0 0 1</fdir> -->
+            <!-- <fdir>0 0 0</fdir> -->
             <!-- <kp value="${kp}" /> -->
             <!-- <kd value="10" /> -->
@@ -302,5 +200,5 @@
               <mechanicalReduction>1</mechanicalReduction>
             </actuator>
-            <joint name="body_to_joint_1_${leg_posi}">
+            <joint name="joint_1_${leg_posi}">
                 <hardwareInterface>hardware_interface/EffortJointInterface</hardwareInterface>
             </joint>
@@ -312,5 +210,5 @@
                 <mechanicalReduction>1</mechanicalReduction>
             </actuator>
-            <joint name="joint_1_${leg_posi}_to_joint_2_${leg_posi}">
+            <joint name="joint_2_${leg_posi}">
                 <hardwareInterface>hardware_interface/EffortJointInterface</hardwareInterface>
             </joint>
@@ -322,5 +220,5 @@
                 <mechanicalReduction>1</mechanicalReduction>
             </actuator>
-            <joint name="link_2_${leg_posi}_to_joint_3_${leg_posi}">
+            <joint name="joint_3_${leg_posi}">
                 <hardwareInterface>hardware_interface/EffortJointInterface</hardwareInterface>
             </joint>
@@ -332,5 +230,5 @@
                 <mechanicalReduction>1</mechanicalReduction>
             </actuator>
-            <joint name="link_3_${leg_posi}_to_joint_4_${leg_posi}">
+            <joint name="joint_4_${leg_posi}">
                 <hardwareInterface>hardware_interface/EffortJointInterface</hardwareInterface>
             </joint>

File: src/rollerwalker_sim/xacro/include/rollerwalker_macro.xacro (robot description, xacro)
@@ -103,5 +103,5 @@
     <xacro:property name="I_link_4_zz" value="${1/12*link_4_mass*(link_4_x*link_4_x + link_4_y*link_4_y)}" />   <!--1/12m(w^2+d^2)-->
     <!-- ジョイントのダンピング係数 -->
-    <xacro:property name="body_to_joint_1_damping"    value="0.1" />   <!-- ボディーからジョイント1のダンピング係数 -->
+    <xacro:property name="joint_1_damping"    value="0.1" />   <!-- ボディーからジョイント1のダンピング係数 -->
     <xacro:property name="joint_1_to_joint_2_damping" value="0.1" />   <!-- ジョイント1からジョイント2のダンピング係数 -->
     <xacro:property name="joint_2_to_link_2_damping"  value="0.1" />   <!-- ジョイント2からリンク2のダンピング係数 -->
