Commit message: 12/6

File: src/rollerwalker_sim/xacro/include/leg_macro.xacro (robot description, xacro)
@@ -188,7 +188,19 @@
         <gazebo reference="wheel_${leg_posi}">
             <material>Gazebo/Blue</material>
-            <mu1>${mu_1}</mu1>
+            <mu>${mu}</mu>
             <mu2>${mu_2}</mu2>
-            <!-- <fdir>0 0 0</fdir> -->
+            <fdir>0 0 1</fdir>
+            <!-- <xacro:if value="${leg_posi=='lf'}">
+                <fdir>1 0 0</fdir>
+            </xacro:if>
+            <xacro:if value="${leg_posi=='lr'}">
+                <fdir>1 0 0</fdir>
+            </xacro:if>
+            <xacro:if value="${leg_posi=='rr'}">
+                <fdir>-1 0 0</fdir>
+            </xacro:if>
+            <xacro:if value="${leg_posi=='rf'}">
+                <fdir>-1 0 0</fdir>
+            </xacro:if> -->
             <!-- <kp value="${kp}" /> -->
             <!-- <kd value="10" /> -->
@@ -241,5 +253,5 @@
             </actuator>
             <joint name="link_4_${leg_posi}_to_wheel_${leg_posi}">
-                <hardwareInterface>hardware_interface/VelocityJointInterface</hardwareInterface>
+                <hardwareInterface>hardware_interface/EffortJointInterface</hardwareInterface>
             </joint>
         </transmission>

File: src/rollerwalker_sim/xacro/include/rollerwalker_macro.xacro (robot description, xacro)
@@ -112,7 +112,7 @@
     <xacro:property name="link_4_to_wheel_damping"    value="0.1" />   <!-- リンク4からホイールのダンピング係数 -->
         <!-- 摩擦力 -->
-    <!-- <xacro:property name="mu_1" value="0.417" />
+    <!-- <xacro:property name="mu" value="0.417" />
     <xacro:property name="mu_2" value="0.0264" />    -->
-    <xacro:property name="mu_1" value="0.417" />
+    <xacro:property name="mu" value="0.0264" />
     <xacro:property name="mu_2" value="0.417" />
     <!-- めり込み係数 -->

Commit message: modify first_pose

File: src/rollerwalker_sim/xacro/include/leg_macro.xacro (robot description, xacro)
@@ -10,20 +10,20 @@
             <!-- lf -->
             <xacro:if value="${leg_posi=='lf'}">
-                <origin xyz="${body_length/2 - joint_1_radius/2} ${body_width/2 - joint_1_radius/2} 0.0" rpy="0 0 0"/>
+                <origin xyz="${body_length/2 - joint_1_radius/2} ${body_width/2 - joint_1_radius/2} 0.0" rpy="0 0 1.5708"/>
                 <limit lower="0.2" upper="3" effort="${effort_limit}" velocity="100"/>
             </xacro:if>
             <!-- lr -->
             <xacro:if value="${leg_posi=='lr'}">
-                <origin xyz="${-(body_length/2 - joint_1_radius/2)} ${body_width/2 - joint_1_radius/2} 0.0" rpy="0 0 0"/>
+                <origin xyz="${-(body_length/2 - joint_1_radius/2)} ${body_width/2 - joint_1_radius/2} 0.0" rpy="0 0 1.5708"/>
                 <limit lower="0.2" upper="3" effort="${effort_limit}" velocity="100"/>
             </xacro:if>
             <!-- rr -->
             <xacro:if value="${leg_posi=='rr'}">
-                <origin xyz="${-(body_length/2 - joint_1_radius/2)} ${-(body_width/2 - joint_1_radius/2)} 0.0" rpy="0 0 0"/>
+                <origin xyz="${-(body_length/2 - joint_1_radius/2)} ${-(body_width/2 - joint_1_radius/2)} 0.0" rpy="0 0 -1.5708"/>
                 <limit lower="-3" upper="-0.2" effort="${effort_limit}" velocity="100"/>
             </xacro:if>
             <!-- rf -->
             <xacro:if value="${leg_posi=='rf'}">
-                <origin xyz="${body_length/2 - joint_1_radius/2} ${-(body_width/2 - joint_1_radius/2)} 0.0" rpy="0 0 0"/>
+                <origin xyz="${body_length/2 - joint_1_radius/2} ${-(body_width/2 - joint_1_radius/2)} 0.0" rpy="0 0 -1.5708"/>
                 <limit lower="-3" upper="-0.2" effort="${effort_limit}" velocity="100"/>
             </xacro:if>
@@ -93,5 +93,5 @@
             <parent link="link_2_${leg_posi}"/>
             <child  link="link_3_${leg_posi}"/>
-            <origin rpy="0 0 0" xyz="${link_2_x} 0 0"/>
+            <origin rpy="0 1.5708 0" xyz="${link_2_x} 0 0"/>
             <dynamics damping="${link_2_to_joint_3_damping}"/>
             <limit lower="-2.0" upper="1.5" effort="${effort_limit}" velocity="100"/>
@@ -190,5 +190,5 @@
             <mu>${mu}</mu>
             <mu2>${mu_2}</mu2>
-            <fdir>0 0 1</fdir>
+            <!-- <fdir>0 0 1</fdir> -->
             <!-- <xacro:if value="${leg_posi=='lf'}">
                 <fdir>1 0 0</fdir>

File: src/rollerwalker_sim/xacro/include/rollerwalker_macro.xacro (robot description, xacro)
@@ -112,8 +112,8 @@
     <xacro:property name="link_4_to_wheel_damping"    value="0.1" />   <!-- リンク4からホイールのダンピング係数 -->
         <!-- 摩擦力 -->
-    <!-- <xacro:property name="mu" value="0.417" />
-    <xacro:property name="mu_2" value="0.0264" />    -->
-    <xacro:property name="mu" value="0.0264" />
-    <xacro:property name="mu_2" value="0.417" />
+    <xacro:property name="mu" value="0.417" />
+    <xacro:property name="mu_2" value="0.0264" />
+    <!-- <xacro:property name="mu" value="0.0264" />
+    <xacro:property name="mu_2" value="0.417" />     -->
     <!-- めり込み係数 -->
     <xacro:property name="kp" value="100000" />

File: src/rollerwalker_sim/xacro/rollerwalker.xacro (robot description, xacro)
@@ -2,9 +2,11 @@
     <xacro:include filename="$(find rollerwalker_sim)/xacro/include/leg_macro.xacro" />
     <!-- 本体の描画 -->
-    <link name="base_link"/>
+    <link name="base_link">
+        <origin xyz="0 0 ${body_z}" rpy="0 0 0"/>
+    </link>
     <joint name="base_to_body" type="fixed">
         <parent link="base_link"/>
         <child  link="body"/>
-        <origin xyz="0 0 ${body_z}" rpy="0 0 0"/>
+        <origin xyz="0 0 0" rpy="0 0 0"/>
     </joint>
     <!-- ボディ -->

Commit message: complete basic rollerwalker gazebo model

File: src/rollerwalker_sim/xacro/include/leg_macro.xacro (robot description, xacro)
@@ -11,21 +11,18 @@
             <xacro:if value="${leg_posi=='lf'}">
                 <origin xyz="${body_length/2 - joint_1_radius/2} ${body_width/2 - joint_1_radius/2} 0.0" rpy="0 0 1.5708"/>
-                <limit lower="0.2" upper="3" effort="${effort_limit}" velocity="100"/>
             </xacro:if>
             <!-- lr -->
             <xacro:if value="${leg_posi=='lr'}">
                 <origin xyz="${-(body_length/2 - joint_1_radius/2)} ${body_width/2 - joint_1_radius/2} 0.0" rpy="0 0 1.5708"/>
-                <limit lower="0.2" upper="3" effort="${effort_limit}" velocity="100"/>
             </xacro:if>
             <!-- rr -->
             <xacro:if value="${leg_posi=='rr'}">
                 <origin xyz="${-(body_length/2 - joint_1_radius/2)} ${-(body_width/2 - joint_1_radius/2)} 0.0" rpy="0 0 -1.5708"/>
-                <limit lower="-3" upper="-0.2" effort="${effort_limit}" velocity="100"/>
             </xacro:if>
             <!-- rf -->
             <xacro:if value="${leg_posi=='rf'}">
                 <origin xyz="${body_length/2 - joint_1_radius/2} ${-(body_width/2 - joint_1_radius/2)} 0.0" rpy="0 0 -1.5708"/>
-                <limit lower="-3" upper="-0.2" effort="${effort_limit}" velocity="100"/>
-            </xacro:if>
+            </xacro:if>
+            <limit lower="-0.4" upper="0.4" effort="${effort_limit}" velocity="100"/>
             <dynamics damping="${joint_1_damping}"/>
         </joint>
@@ -162,5 +159,5 @@
             <child  link="wheel_${leg_posi}"/>
             <origin rpy="0 1.57070 0" xyz="${link_4_x + wheel_thickness/2} 0 0"/>
-            <dynamics damping="${link_4_to_wheel_damping}"/>
+            <dynamics damping="${link_4_to_wheel_damping}" />
             <!-- <limit lower="-1.79769e+308" upper="1.79769e+308" effort="0" velocity="0"/> -->
         </joint>
@@ -188,21 +185,9 @@
         <gazebo reference="wheel_${leg_posi}">
             <material>Gazebo/Blue</material>
-            <mu>${mu}</mu>
+            <mu1>${mu}</mu1>
             <mu2>${mu_2}</mu2>
-            <!-- <fdir>0 0 1</fdir> -->
-            <!-- <xacro:if value="${leg_posi=='lf'}">
-                <fdir>1 0 0</fdir>
-            </xacro:if>
-            <xacro:if value="${leg_posi=='lr'}">
-                <fdir>1 0 0</fdir>
-            </xacro:if>
-            <xacro:if value="${leg_posi=='rr'}">
-                <fdir>-1 0 0</fdir>
-            </xacro:if>
-            <xacro:if value="${leg_posi=='rf'}">
-                <fdir>-1 0 0</fdir>
-            </xacro:if> -->
-            <!-- <kp value="${kp}" /> -->
-            <!-- <kd value="10" /> -->
+            <fdir1>1 0 0</fdir1>
+            <!-- <kp value="0.0001" />
+            <kd value="0.2" /> -->
         </gazebo>
         <!-- トランスミッション -->

File: src/rollerwalker_sim/xacro/include/rollerwalker_macro.xacro (robot description, xacro)
@@ -110,8 +110,8 @@
     <xacro:property name="link_3_to_joint_4_damping"  value="0.1" />   <!-- リンク3からジョイント4のダンピング係数 -->
     <xacro:property name="joint_4_to_link_4_damping"  value="0.1" />   <!-- ジョイント4からリンク4のダンピング係数 -->
-    <xacro:property name="link_4_to_wheel_damping"    value="0.1" />   <!-- リンク4からホイールのダンピング係数 -->
+    <xacro:property name="link_4_to_wheel_damping"    value="0.01" />   <!-- リンク4からホイールのダンピング係数 -->
         <!-- 摩擦力 -->
     <xacro:property name="mu" value="0.417" />
-    <xacro:property name="mu_2" value="0.0264" />
+    <xacro:property name="mu_2" value="0.417" />
     <!-- <xacro:property name="mu" value="0.0264" />
     <xacro:property name="mu_2" value="0.417" />     -->

Commit message: modify leg cordinate

File: src/rollerwalker_sim/xacro/include/leg_macro.xacro (robot description, xacro)
@@ -10,9 +10,9 @@
             <!-- lf -->
             <xacro:if value="${leg_posi=='lf'}">
-                <origin xyz="${body_length/2 - joint_1_radius/2} ${body_width/2 - joint_1_radius/2} 0.0" rpy="0 0 1.5708"/>
+                <origin xyz="${body_length/2 - joint_1_radius/2} ${body_width/2 - joint_1_radius/2} 0.0" rpy="0 3.141519 -1.5708"/>
             </xacro:if>
             <!-- lr -->
             <xacro:if value="${leg_posi=='lr'}">
-                <origin xyz="${-(body_length/2 - joint_1_radius/2)} ${body_width/2 - joint_1_radius/2} 0.0" rpy="0 0 1.5708"/>
+                <origin xyz="${-(body_length/2 - joint_1_radius/2)} ${body_width/2 - joint_1_radius/2} 0.0" rpy="0 3.141519 -1.5708"/>
             </xacro:if>
             <!-- rr -->
@@ -57,5 +57,16 @@
             <parent link="joint_1_link_${leg_posi}"/>
             <child  link="link_2_${leg_posi}"/>
-            <origin rpy="0 0 0" xyz="0 0 0"/>
+            <xacro:if value="${leg_posi=='lf'}">
+                <origin rpy="3.141519 0 0" xyz="0 0 0"/>
+            </xacro:if>
+            <xacro:if value="${leg_posi=='lr'}">
+                <origin rpy="3.141519 0 0" xyz="0 0 0"/>
+            </xacro:if>
+            <xacro:if value="${leg_posi=='rr'}">
+                <origin rpy="0 0 0" xyz="0 0 0"/>
+            </xacro:if>
+            <xacro:if value="${leg_posi=='rf'}">
+                <origin rpy="0 0 0" xyz="0 0 0"/>
+            </xacro:if>
             <dynamics damping="${joint_1_to_joint_2_damping}"/>
             <limit lower="-1.5" upper="1.5" effort="${effort_limit}" velocity="100"/>
@@ -124,5 +135,5 @@
             <parent link="link_3_${leg_posi}"/>
             <child  link="link_4_${leg_posi}"/>
-            <origin rpy="0 0 0" xyz="${link_3_x} 0 0"/>
+            <origin rpy="0 -1.57070 0" xyz="${link_3_x} 0 0"/>
             <dynamics damping="${link_3_to_joint_4_damping}"/>
             <limit lower="-2.0" upper="1.5" effort="${effort_limit}" velocity="100"/>

Commit message: 12/18

File: src/rollerwalker_sim/xacro/include/leg_macro.xacro (robot description, xacro)
@@ -135,5 +135,5 @@
             <parent link="link_3_${leg_posi}"/>
             <child  link="link_4_${leg_posi}"/>
-            <origin rpy="0 -1.57070 0" xyz="${link_3_x} 0 0"/>
+            <origin rpy="0 0 0" xyz="${link_3_x} 0 0"/>
             <dynamics damping="${link_3_to_joint_4_damping}"/>
             <limit lower="-2.0" upper="1.5" effort="${effort_limit}" velocity="100"/>

Commit message: setup PID paramator

File: src/rollerwalker_sim/xacro/include/leg_macro.xacro (robot description, xacro)
@@ -137,5 +137,5 @@
             <origin rpy="0 0 0" xyz="${link_3_x} 0 0"/>
             <dynamics damping="${link_3_to_joint_4_damping}"/>
-            <limit lower="-2.0" upper="1.5" effort="${effort_limit}" velocity="100"/>
+            <limit lower="-2.0" upper="2.0" effort="${effort_limit}" velocity="100"/>
         </joint>
         <link name = "link_4_${leg_posi}">
