Commit message: make velocity publisher

File: src/rollerwalker_sim/xacro/include/rollerwalker_macro.xacro (robot description, xacro)
@@ -110,5 +110,5 @@
     <xacro:property name="link_3_to_joint_4_damping"  value="0.1" />   <!-- リンク3からジョイント4のダンピング係数 -->
     <xacro:property name="joint_4_to_link_4_damping"  value="0.1" />   <!-- ジョイント4からリンク4のダンピング係数 -->
-    <xacro:property name="link_4_to_wheel_damping"    value="0.01" />   <!-- リンク4からホイールのダンピング係数 -->
+    <xacro:property name="link_4_to_wheel_damping"    value="0.005" />   <!-- リンク4からホイールのダンピング係数 -->
         <!-- 摩擦力 -->
     <xacro:property name="mu" value="0.417" />
@@ -120,3 +120,5 @@
     <!-- effort_limit -->
     <xacro:property name="effort_limit" value="100000" />
+    <!-- gazebo上の位置のパブリッシュレート -->
+    <xacro:property name="gazebo_position_publish_rate" value="50" />
 </robot>

File: src/rollerwalker_sim/xacro/rollerwalker.xacro (robot description, xacro)
@@ -45,4 +45,10 @@
             <legacyModeNS>true</legacyModeNS>
         </plugin>
+        <plugin name="ground_truth" filename="libgazebo_ros_p3d.so">
+            <frameName>world</frameName>
+            <bodyName>base_link</bodyName>
+            <topicName>/true_position</topicName>
+            <updateRate>${gazebo_position_publish_rate}</updateRate>
+        </plugin>
     </gazebo>
 </robot>

Commit message: 12/19 complete calZ

File: src/rollerwalker_sim/xacro/include/rollerwalker_macro.xacro (robot description, xacro)
@@ -40,5 +40,5 @@
     <!-- 各リンクの長さ -->
     <xacro:property name="l2" value="0.2" />
-    <xacro:property name="l3" value="0.243" />
+    <xacro:property name="l3" value="0.188" />
     <xacro:property name="l4" value="0.031" />
     <!-- タイヤ関連 -->
@@ -79,5 +79,5 @@
     <!-- 各足の長さはlink_n_xの値を変えれば良い -->
     <!-- リンク2関連 -->
-    <xacro:property name="link_2_x" value="0.2" />
+    <xacro:property name="link_2_x" value="${l2}" />
     <xacro:property name="link_2_y" value="0.055" />
     <xacro:property name="link_2_z" value="0.09" />
@@ -87,5 +87,5 @@
     <xacro:property name="I_link_2_zz" value="${1/12*link_2_mass*(link_2_x*link_2_x + link_2_y*link_2_y)}" />   <!--1/12m(w^2+d^2)-->
     <!-- リンク3関連 -->
-    <xacro:property name="link_3_x" value="0.188" />
+    <xacro:property name="link_3_x" value="${l3}" />
     <xacro:property name="link_3_y" value="0.045" />
     <xacro:property name="link_3_z" value="0.049" />
@@ -95,7 +95,7 @@
     <xacro:property name="I_link_3_zz" value="${1/12*link_3_mass*(link_3_x*link_3_x + link_3_y*link_3_y)}" />   <!--1/12m(w^2+d^2)-->
     <!-- リンク4関連 -->
-    <xacro:property name="link_4_x" value="0.044" />
+    <xacro:property name="link_4_x" value="${l4}" />
     <xacro:property name="link_4_y" value="0.043" />
-    <xacro:property name="link_4_z" value="0.031" />
+    <xacro:property name="link_4_z" value="0.044" />
     <!-- リンク4のイナーシャ -->
     <xacro:property name="I_link_4_xx" value="${1/12*link_4_mass*(link_4_y*link_4_y + link_4_z*link_4_z)}" />   <!--1/12m(h^2+d^2)-->

Commit message: make time reset

File: src/rollerwalker_sim/xacro/include/rollerwalker_macro.xacro (robot description, xacro)
@@ -119,4 +119,4 @@
     <xacro:property name="effort_limit" value="100000" />
     <!-- gazebo上の位置のパブリッシュレート -->
-    <xacro:property name="gazebo_position_publish_rate" value="50" />
+    <xacro:property name="gazebo_position_publish_rate" value="100" />
 </robot>
