Commit message: 1/14

File: src/rollerwalker_sim/xacro/include/gazebo_plugin.xacro (robot description, xacro)
@@ -31,5 +31,5 @@
                 <link>rollerwalker::wheel_lr</link>     <!--リンク名-->
                 <pose>0 0 0 0 0 0</pose>                <!--プロット位置（フレームからの位置）-->
-                <material>Gazebo/Red</material>         <!--プロットの色-->
+                <material>Gazebo/Green</material>         <!--プロットの色-->
             </plot>
             <!-- 右後ろタイヤの軌跡 -->
@@ -37,5 +37,5 @@
                 <link>rollerwalker::wheel_rr</link>     <!--リンク名-->
                 <pose>0 0 0 0 0 0</pose>                <!--プロット位置（フレームからの位置）-->
-                <material>Gazebo/Red</material>         <!--プロットの色-->
+                <material>Gazebo/Green</material>         <!--プロットの色-->
             </plot>
             <!-- 右前タイヤの軌跡 -->

File: src/rollerwalker_sim/xacro/include/leg_macro.xacro (robot description, xacro)
@@ -24,5 +24,5 @@
                 <origin xyz="${body_length/2 - joint_1_radius/2} ${-(body_width/2 - joint_1_radius/2)} 0.0" rpy="0 0 -1.5708"/>
             </xacro:if>
-            <limit lower="-0.4" upper="0.4" effort="${effort_limit}" velocity="100"/>
+            <limit lower="-1.5" upper="1.5" effort="${effort_limit}" velocity="100"/>
             <dynamics damping="${joint_1_damping}"/>
         </joint>

Commit message: delete file writer

File: src/rollerwalker_sim/xacro/include/gazebo_plugin.xacro (robot description, xacro)
@@ -12,38 +12,4 @@
             <updateRate>${gazebo_position_publish_rate}</updateRate>
         </plugin>
-        <plugin name='3dplot' filename='libLinkPlot3DPlugin.so'>
-            <!-- Update at 10 Hz -->
-            <frequency>10</frequency>
-            <!-- 本体リンクの軌跡 -->
-            <plot>
-                <link>rollerwalker::base_link</link>    <!--リンク名-->
-                <pose>0 0 0 0 0 0</pose>                <!--プロット位置（フレームからの位置）-->
-                <material>Gazebo/Blue</material>        <!--プロットの色-->
-            </plot>
-            <!-- 左前タイヤの軌跡 -->
-            <plot>
-                <link>rollerwalker::wheel_lf</link>     <!--リンク名-->
-                <pose>0 0 0 0 0 0</pose>                <!--プロット位置（フレームからの位置）-->
-                <material>Gazebo/Red</material>         <!--プロットの色-->
-            </plot>
-            <!-- 左後ろタイヤの軌跡 -->
-            <plot>
-                <link>rollerwalker::wheel_lr</link>     <!--リンク名-->
-                <pose>0 0 0 0 0 0</pose>                <!--プロット位置（フレームからの位置）-->
-                <material>Gazebo/Green</material>         <!--プロットの色-->
-            </plot>
-            <!-- 右後ろタイヤの軌跡 -->
-            <plot>
-                <link>rollerwalker::wheel_rr</link>     <!--リンク名-->
-                <pose>0 0 0 0 0 0</pose>                <!--プロット位置（フレームからの位置）-->
-                <material>Gazebo/Green</material>         <!--プロットの色-->
-            </plot>
-            <!-- 右前タイヤの軌跡 -->
-            <plot>
-                <link>rollerwalker::wheel_rf</link>     <!--リンク名-->
-                <pose>0 0 0 0 0 0</pose>                <!--プロット位置（フレームからの位置）-->
-                <material>Gazebo/Red</material>         <!--プロットの色-->
-            </plot>
-        </plugin>
     </gazebo>
 </robot>
